File: Relay_board/Relay_board.kicad_sch (KiCad schematic)
At the start: 43 parts, among them J1 AC_Power_out, J2 Earth_Out, J3 AC_In, J4 DC_Relay_In, J5 Control, K1 G5LE-1-DC5, K2 G5LE-1-DC12, K3 G5LE-1-DC12, Q1 S8050, Q2 S8050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

Commit message: Fixed AC paths
Connections:
- net AC_Line_1 is gone; now on net Live: J1.1 (Pin_1)
- net AC_Line_2 is gone; now on net Neutral: J1.2 (Pin_2)
- net Live: now also PS1.2 (AC/L); no longer PS1.1 (AC/N)
- net Neutral: now also J3.2 (Pin_2), PS1.1 (AC/N)
- removed net Nutral: J3.2 (Pin_2), PS1.2 (AC/L)
Changed lines of the file:
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@@
     (effects (font (size 1.27 1.27)) (justify left bottom))
   )
-  (label "Nutral" (at 63.5 82.55 0)
+  (label "Live" (at 63.5 82.55 0)
     (effects (font (size 1.27 1.27)) (justify left bottom))
   )
@@
     (effects (font (size 1.27 1.27)) (justify left bottom))
   )
-  (label "AC_Line_1" (at 335.28 134.62 0)
+  (label "Live" (at 335.28 134.62 0)
     (effects (font (size 1.27 1.27)) (justify left bottom))
   )
@@
     (effects (font (size 1.27 1.27)) (justify left bottom))
   )
-  (label "Live" (at 63.5 87.63 0)
+  (label "Neutral" (at 63.5 87.63 0)
     (effects (font (size 1.27 1.27)) (justify left bottom))
   )
-  (label "Nutral" (at 364.49 30.48 270)
+  (label "Neutral" (at 364.49 30.48 270)
     (effects (font (size 1.27 1.27)) (justify right bottom))
   )
@@
     (effects (font (size 1.27 1.27)) (justify left bottom))
   )
-  (label "Nutral" (at 335.28 166.37 0)
+  (label "Neutral" (at 335.28 166.37 0)
     (effects (font (size 1.27 1.27)) (justify left bottom))
   )
@@
     (effects (font (size 1.27 1.27)) (justify left bottom))
   )
-  (label "AC_Line_2" (at 335.28 137.16 0)
+  (label "Neutral" (at 335.28 137.16 0)
     (effects (font (size 1.27 1.27)) (justify left bottom))
   )
